Commit message: reduced drive wheel height offset to 0.5mm

File: omron_ld60_description/models/LD60_no_castors.xacro (robot description, xacro)
@@ -25,5 +25,5 @@
   <xacro:property name="axis_offset" value="0.025"/>
   <xacro:property name="wheel_collision_scaler" value="0.01"/>
-  <xacro:property name="drive_wheel_height_offset" value="0.001"/>
+  <xacro:property name="drive_wheel_height_offset" value="0.0005"/>
   <!-- extra links + joints for castors -->
   <xacro:macro name="castor_base" params="name parent xyz">

Commit message: modified no castors model

File: omron_ld60_description/models/LD60_no_castors.xacro (robot description, xacro)
@@ -25,5 +25,5 @@
   <xacro:property name="axis_offset" value="0.025"/>
   <xacro:property name="wheel_collision_scaler" value="0.01"/>
-  <xacro:property name="drive_wheel_height_offset" value="0.0005"/>
+  <xacro:property name="drive_wheel_height_offset" value="0.001"/>
   <!-- extra links + joints for castors -->
   <xacro:macro name="castor_base" params="name parent xyz">
@@ -152,4 +152,27 @@
   <xacro:castor_wheel name="lb_castor_wheel" parent="lb_castor_base" xyz="-${axis_offset} 0 0"/>
   <xacro:castor_wheel name="rb_castor_wheel" parent="rb_castor_base" xyz="-${axis_offset} 0 0"/>
+  <!-- Lidar Frames -->
+  <link name="lower_laser">
+    <inertial>
+      <mass value="0.001"/>
+      <inertia ixx="0.0000001" ixy="0.0" ixz="0.0" iyy="0.0000001" iyz="0.0" izz="0.0000001"/>
+    </inertial>
+  </link>
+  <link name="upper_laser">
+    <inertial>
+      <mass value="0.001"/>
+      <inertia ixx="0.0000001" ixy="0.0" ixz="0.0" iyy="0.0000001" iyz="0.0" izz="0.0000001"/>
+    </inertial>
+  </link>
+  <joint name="main_body_to_upper_laser" type="fixed">
+    <parent link="main_body"/>
+    <child link="upper_laser"/>
+    <origin xyz="0.27 0 0.11"/>
+  </joint>
+  <joint name="main_body_to_lower_laser" type="fixed">
+    <parent link="main_body"/>
+    <child link="lower_laser"/>
+    <origin xyz="0.27 0 -0.03"/>
+  </joint>
   <gazebo reference="right_wheel">
     <material>Gazebo/Black</material>
